File: Schematics/Power.kicad_sch (KiCad schematic)
At the start: 0 parts

Commit message: Need to order stencil
Parts:
- added C3, C4: 1000uF, Capacitor_SMD:CP_Elec_8x6.9, symbol Device:C_Polarized_Small_US
- added D9: D_Schottky, Diode_SMD:D_0805_2012Metric, symbol Device:D_Schottky_Small
- added H1, H2, H3, H4: MountingHole, MountingHole:MountingHole_3mm, symbol Mechanical:MountingHole
- added J12: USB_C_Receptacle, UE_USB:USB_C_Receptical-Jing, symbol Connector:USB_C_Receptacle
- added J13: Power, TerminalBlock:TerminalBlock_bornier-2_P5.08mm, symbol Connector_Generic:Conn_01x02
- added L3: 100uH, Inductor_SMD:L_Sunlord_MWSA1205S-R50, symbol Device:L_Small
- added RN4: 5.1k, Resistor_SMD:R_Array_Concave_4x0603, symbol Device:R_Pack04
- added U2: LM2576S-3.3, Package_TO_SOT_SMD:TO-263-5_TabPin3, symbol Regulator_Switching:LM2576S-3.3
Connections:
- new net: D9.1 (K), L3.1, U2.2 (OUT)
- new net: J12.B5 (CC2), RN4.1 (R1.1)
- new net: J12.A5 (CC1), RN4.2 (R2.1)
- new net +5V: C3.1, J12.A4 (VBUS), J12.A9 (VBUS), J12.B4 (VBUS), J12.B9 (VBUS), J13.1 (Pin_1), U2.1 (VIN)
- new net D+: J12.A6 (D+), J12.B6 (D+)
- new net D-: J12.A7 (D-), J12.B7 (D-)
- new net VCC: C4.1, L3.2, U2.4 (FB)
- new net VSS: C3.2, C4.2, D9.2 (A), J12.A1 (GND), J12.A12 (GND), J12.B1 (GND), J12.B12 (GND), J12.S1 (SHIELD), J13.2 (Pin_2), U2.3 (GND), U2.5 (~{ON}/OFF)
- no-connect marks 0 -> 14
