File: Schematics/RPi_CM4.kicad_sch (KiCad schematic)
At the start: 31 parts, among them J1 690-019-298-412, J2 Micro_SD_Card_Det, J3 THD-02-R, J4 Conn_01x03, J5 Conn_02x07_Odd_Even, J6 THD-20-R, U1 RT9742SNGV, U2 RT9742GGJ5, U3 TPD4EUSB30, U4 TPD4EUSB30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

Commit message: Need to order stencil
Parts:
- removed C3: 10u, Capacitor_SMD:C_0805_2012Metric, symbol Device:C
- removed C4: 100n, Capacitor_SMD:C_0402_1005Metric, symbol Device:C
- removed D1: LED Green, LED_SMD:LED_0603_1608Metric, symbol Device:LED
- removed J2: Micro_SD_Card_Det, CM4IO:SDCARD_MOLEX_503398-1892, symbol Connector:Micro_SD_Card_Det
- removed J3: THD-02-R, Connector_PinHeader_2.54mm:PinHeader_2x02_P2.54mm_Vertical, symbol Connector_Generic:Conn_02x02_Odd_Even
- removed R1, R2: nf, Resistor_SMD:R_0402_1005Metric, symbol Device:R
- removed R3: 12K 1%, Resistor_SMD:R_0402_1005Metric, symbol Device:R
- removed R4, R5: 470R, Resistor_SMD:R_0402_1005Metric, symbol Device:R
- removed R6: 1k, Resistor_SMD:R_0402_1005Metric, symbol Device:R
- removed R8: 0R, Resistor_SMD:R_0805_2012Metric_Pad1.15x1.40mm_HandSolder, symbol Device:R
- removed R9: nf, Resistor_SMD:R_0805_2012Metric_Pad1.15x1.40mm_HandSolder, symbol Device:R
- removed TP1: TestPoint, TestPoint:TestPoint_Pad_2.0x2.0mm, symbol Connector:TestPoint
- removed U2: RT9742GGJ5, Package_TO_SOT_SMD:SOT-23-5, symbol CM4IO:RT9742GGJ5
- removed U3, U4: TPD4EUSB30, Package_SON:USON-10_2.5x1.0mm_P0.5mm, symbol CM4IO:TPD4EUSB30
- removed U5: MagJack-A70-112-331N126, CM4IO:TRJG0926HENL, symbol CM4IO:MagJack-A70-112-331N126
- added J14: Conn_01x01, Connector_PinHeader_2.54mm:PinHeader_1x01_P2.54mm_Vertical, symbol Connector_Generic:Conn_01x01
- C1, C2: footprint Capacitor_SMD:C_0402_1005Metric -> Capacitor_SMD:C_0805_2012Metric
- D2: footprint LED_SMD:LED_0603_1608Metric -> LED_SMD:LED_0805_2012Metric
- R7: footprint Resistor_SMD:R_0402_1005Metric -> Resistor_SMD:R_0805_2012Metric
- TP2: footprint TestPoint:TestPoint_Pad_2.0x2.0mm -> TestPoint:TestPoint_THTPad_D1.0mm_Drill0.5mm
Connections:
- net GPIO_VREF is gone; now on net +3.3v: Module1.78 (GPIO_VREF(1.8v/3.3v_Input))
- net GND renamed VSS
- net GPIO10 renamed iCE_MOSI
- net GPIO11 renamed iCE_SCK
- net GPIO14 renamed Serial_RX
- net GPIO15 renamed Serial_TX
- net GPIO8 renamed iCE_SS_B
- net GPIO9 renamed iCE_MISO
- net USB2_N renamed D-
- net USB2_P renamed D+
- net USBOTG_ID: no longer names the net of Module1.101 (USB_OTG_ID)
- net USBOTG_ID: now also J14.1 (Pin_1)
- no-connect marks 10 -> 9
Other:
- note removed: "CM4Lite SDCARD I/F"
- note removed: "Ethernet"
- note removed: "Ethernet POE Protection"
- note removed: "POE Header"
